Commit message: first urdf - draft

File: vulcano_base_description/robots/vulcano_base.urdf.xacro (robot description, xacro)
@@ -5,8 +5,8 @@
 	<!-- ***************** -->
 	<!-- First we import all posible elements defined in the urdf.xacro files. All these elements are defined as macro:xacros -->
-	<!-- Import summit XL base elements -->
+	<!-- Import vulcano base elements -->
 	<xacro:include filename="$(find vulcano_base_description)/urdf/bases/vulcano_base.urdf.xacro" />
 	<!-- Import vulcano wheels -->
-	<!-- xacro:include filename="$(find vulcano_base_description)/urdf/wheels/motor_wheel.urdf.xacro" / -->
+	<xacro:include filename="$(find vulcano_base_description)/urdf/wheels/motor_wheel.urdf.xacro" />
 	<!-- Import all available sensors -->
 	<xacro:include filename="$(find robotnik_sensors)/urdf/all_sensors.urdf.xacro" />
@@ -16,6 +16,6 @@
 	<xacro:property name="PI" value="3.1415926535897931"/>
 	<!-- Wheel parameters -->
-	<xacro:property name="wheel_offset_x" value="0.22911" />    <!-- x,y,z in translation from base_link to the center of the wheel -->
-	<xacro:property name="wheel_offset_y" value="0.24070" />
+	<xacro:property name="wheel_offset_x" value="0.467" />    <!-- x,y,z in translation from base_link to the center of the wheel -->
+	<xacro:property name="wheel_offset_y" value="0.285" />
 	<xacro:property name="wheel_offset_z" value="0.0" />
 	<!-- Flag to select the high or low quality model -->
@@ -30,39 +30,29 @@
   <xacro:ros_control/>
   <!-- Gazebo omni steering plugin -->
-  <!-- xacro:omni_steering/>
-	<xacro:omni_wheel name="front_right" parent="base_link" reflect="false" hq="true">
-		<origin xyz="${wheel_offset_x} -${wheel_offset_y} ${wheel_offset_z}" rpy="0 0 0"/>
-	</xacro:omni_wheel>
-	<xacro:omni_wheel name="front_left" parent="base_link" reflect="true" hq="true">
-		<origin xyz="${wheel_offset_x} ${wheel_offset_y} ${wheel_offset_z}" rpy="0 0 0"/>
-	</xacro:omni_wheel>
-	<xacro:omni_wheel name="back_left" parent="base_link" reflect="false" hq="true">
-		<origin xyz="-${wheel_offset_x} ${wheel_offset_y} ${wheel_offset_z}" rpy="0 0 0"/>
-	</xacro:omni_wheel>
-	<xacro:omni_wheel name="back_right" parent="base_link" reflect="true" hq="true">
-		<origin xyz="-${wheel_offset_x} -${wheel_offset_y} ${wheel_offset_z}" rpy="0 0 0"/>
-	</xacro:omni_wheel -->
-	<!-- SENSORS -->
+  <!-- xacro:omni_steering/ -->
+  <xacro:motor_wheel name="front_right" parent="base_link" reflect="false" hq="true">
+	<origin xyz="${wheel_offset_x} -${wheel_offset_y} ${wheel_offset_z}" rpy="0 0 0"/>
+  </xacro:motor_wheel>
+  <xacro:motor_wheel name="front_left" parent="base_link" reflect="true" hq="true">
+	<origin xyz="${wheel_offset_x} ${wheel_offset_y} ${wheel_offset_z}" rpy="0 0 0"/>
+  </xacro:motor_wheel>
+  <xacro:motor_wheel name="back_left" parent="base_link" reflect="false" hq="true">
+	<origin xyz="-${wheel_offset_x} ${wheel_offset_y} ${wheel_offset_z}" rpy="0 0 0"/>
+  </xacro:motor_wheel>
+  <xacro:motor_wheel name="back_right" parent="base_link" reflect="true" hq="true">
+	<origin xyz="-${wheel_offset_x} -${wheel_offset_y} ${wheel_offset_z}" rpy="0 0 0"/>
+  </xacro:motor_wheel>
+  <!-- SENSORS see robotnik_sensors for the specific configuration -->
   <!-- Hokuyo laser sensors can be parametized with min_angle and max_angle e.g: -->
   <!--xacro:sensor_hokuyo_utm30lx name="hokuyo_base" parent="base_link" min_angle="2.35" max_angle="-2.35"-->
-	<xacro:sensor_hokuyo_utm30lx name="hokuyo_base" parent="base_link">
-		<origin xyz="0.0 0.0 0.33" rpy="0 0 0"/>
-	</xacro:sensor_hokuyo_utm30lx>
-<!--
-	<xacro:sensor_hokuyo_urg04lx name="hokuyo1" parent="base_link">
-		<origin xyz="-0.1 0.0 0.33" rpy="0 0 0"/>
-	</xacro:sensor_hokuyo_urg04lx>
--->
-<!--
-  <xacro:sensor_hokuyo_ust10lx name="hokuyo_base" parent="base_link">
-		<origin xyz="0.0 0.0 0.33" rpy="0 0 0"/>
-	</xacro:sensor_hokuyo_ust10lx>
--->
-	<xacro:sensor_axis name="camera" parent="base_link">
-		<origin xyz="0.19 0 0.17" rpy="0 ${15*PI/180} 0"/>
-	</xacro:sensor_axis>
-	<xacro:sensor_imu name="imu" parent="base_link">
-		<origin xyz="-0.18 0.0 0.170" rpy="0 0 0"/>
-	</xacro:sensor_imu>
+  <xacro:sensor_hokuyo_utm30lx name="hokuyo_base" parent="base_link">
+	 <origin xyz="0.0 0.0 0.33" rpy="0 0 0"/>
+  </xacro:sensor_hokuyo_utm30lx>
+  <xacro:sensor_axis name="camera" parent="base_link">
+	<origin xyz="0.19 0 0.17" rpy="0 ${15*PI/180} 0"/>
+  </xacro:sensor_axis>
+  <xacro:sensor_imu name="imu" parent="base_link">
+	<origin xyz="-0.18 0.0 0.170" rpy="0 0 0"/>
+  </xacro:sensor_imu>
 <!--
 	<xacro:sensor_kinect name="kinect" parent="base_link">

File: vulcano_base_description/urdf/bases/vulcano_base.urdf.xacro (robot description, xacro)
@@ -17,6 +17,5 @@
     </link>
     <joint name="base_footprint_joint" type="fixed">
-      <!-- origin xyz="0 0 ${wheel_radius}" rpy="0 0 0" / --> <!-- ${wheel_radius} property must be defined inside wheel description -->
-      <origin xyz="0 0 0.15" rpy="0 0 0" />
+      <origin xyz="0 0 ${wheel_radius}" rpy="0 0 0" /> <!-- ${wheel_radius} property must be defined inside wheel description -->
       <parent link="base_footprint"/>
       <child link="base_link" />
@@ -83,5 +82,5 @@
   </link>
   <joint name="cabinet_joint" type="fixed">
-    <origin xyz="0 0 0" rpy="0 0 0" />
+    <origin xyz="0 0 0.234" rpy="0 0 0" />
     <parent link="base_link"/>
     <child link="cabinet_link" />

File: vulcano_base_description/urdf/wheels/motor_wheel.urdf.xacro (robot description, xacro)
@@ -3,7 +3,17 @@
   <xacro:property name="M_PI" value="3.1415926535897931" />
   <!-- Wheels -->
-  <property name="wheel_radius" value="0.117" />
+  <property name="wheel_radius" value="0.093" />
   <property name="wheel_height" value="0.14" />
   <property name="wheel_mass" value="6.5" /> <!-- in kg-->
+  <xacro:property name="steer_joint_damping" value="2.0" />
+  <xacro:property name="steer_joint_friction" value="1.0" />
+  <xacro:property name="steer_joint_effort_limit" value="100.0" />
+  <xacro:property name="steer_joint_velocity_limit" value="100.0" />
+  <xacro:property name="motor_wheel_mechanical_reduction" value="100.0" />
+  <xacro:property name="wheel_joint_damping" value="1.0" />
+  <xacro:property name="wheel_joint_friction" value="1.0" />
+  <xacro:property name="wheel_joint_effort_limit" value="1000.0" />
+  <xacro:property name="wheel_joint_velocity_limit" value="2000.0" />
+  <xacro:property name="wheel_mechanical_reduction" value="1.0" />
   <xacro:macro name="cylinder_inertia" params="m r h">
     <inertia  ixx="${m*(3*r*r+h*h)/12}" ixy = "0" ixz = "0"
@@ -12,14 +22,6 @@
   </xacro:macro>
   <xacro:macro name="motor_wheel" params="name parent *origin reflect hq">
-  <!--WHEEL TIRE -->
-    <joint name="joint_${name}_wheel" type="continuous">
-      <parent link="${parent}"/>
-      <child link="${name}_wheel"/>
-      <insert_block name="origin" />
-      <axis xyz="0 1 0" rpy="0 0 0" />
-      <limit effort="100" velocity="100"/>
-      <joint_properties damping="0.0" friction="0.0"/>
-    </joint>
-    <link name="${name}_wheel">
+  <!--MOTOR WHEEL -->
+  <link name="${name}_motor_wheel">
       <visual>
         <!-- HIGH RESOLUTION WHEELS -->
@@ -27,10 +29,72 @@
           <origin xyz="0 0 0" rpy="0 0 0" />
           <geometry>
-						<xacro:if value="${reflect}">
-							<mesh filename="package://vulcano_base_description/meshes/wheels/rubber_wheel_left.dae" />
-						</xacro:if>
-						<xacro:unless value="${reflect}">
-							<mesh filename="package://summit_xl_description/meshes/wheels/rubber_wheel_right.dae" />
-						</xacro:unless>
+				<xacro:if value="${reflect}">
+					<mesh filename="package://vulcano_base_description/meshes/wheels/motorwheel_2.dae" />
+				</xacro:if>
+				<xacro:unless value="${reflect}">
+					<mesh filename="package://vulcano_base_description/meshes/wheels/motorwheel_2.dae" />
+				</xacro:unless>
+          </geometry>
+        </xacro:if>
+       <!-- LOW RESOLUTION WHEELS -->
+        <xacro:unless value="${hq}">
+          <origin xyz="0 0 0" rpy="0 0 0" />
+          <geometry>
+				<xacro:if value="${reflect}">
+					<mesh filename="package://vulcano_base_description/meshes/wheels/motorwheel_2.stl" />
+				</xacro:if>
+				<xacro:unless value="${reflect}">
+					<mesh filename="package://vulcano_base_description/meshes/wheels/motorwheel_2.stl" />
+				</xacro:unless>
+          </geometry>
+        </xacro:unless>
+      </visual>
+      <collision>
+		<origin xyz="0 0 0" rpy="0 0 0" />
+        <geometry>
+				<xacro:if value="${reflect}">
+					<mesh filename="package://vulcano_base_description/meshes/wheels/motorwheel_2.dae" />
+				</xacro:if>
+				<xacro:unless value="${reflect}">
+					<mesh filename="package://vulcano_base_description/meshes/wheels/motorwheel_2.dae" />
+				</xacro:unless>
+        </geometry>
+      </collision>
+      <inertial>
+        <mass value="20" />
+        <origin xyz="0 0 0" />
+		<inertia  ixx="0.01" ixy="0.0"  ixz="0.0"  iyy="0.01"  iyz="0.0"  izz="0.01" />
+	  </inertial>
+    </link>
+    <joint name="joint_${name}_motor_wheel" type="continuous">
+      <parent link="${parent}"/>
+      <child link="${name}_motor_wheel"/>
+      <insert_block name="origin" />
+      <axis xyz="0 0 1" rpy="0 0 0" />
+      <!-- limit effort="${steer_joint_effort_limit}" velocity="${steer_joint_velocity_limit}" lower="-1.5708" upper="1.5708"/ -->
+      <limit effort="${steer_joint_effort_limit}" velocity="${steer_joint_velocity_limit}" lower="-3.00" upper="3.00"/>
+      <joint_properties damping="${steer_joint_damping}" friction="{steer_joint_friction}"/>
+    </joint>
+  <transmission name="${name}_motor_wheel_joint_trans">
+	 <type>transmission_interface/SimpleTransmission</type>
+     <joint name="joint_${name}_motor_wheel">
+		<hardwareInterface>EffortJointInterface</hardwareInterface>
+     </joint>
+     <actuator name="${name}_motor_wheel_joint_motor">
+        <mechanicalReduction>${motor_wheel_mechanical_reduction}</mechanicalReduction>
+     </actuator>
+  </transmission>
+  <link name="${name}_wheel">
+      <visual>
+        <!-- HIGH RESOLUTION WHEELS -->
+        <xacro:if value="${hq}">
+          <origin xyz="0 0 0" rpy="0 0 0" />
+          <geometry>
+				<xacro:if value="${reflect}">
+					<mesh filename="package://vulcano_base_description/meshes/wheels/wheel_1.dae" />
+				</xacro:if>
+				<xacro:unless value="${reflect}">
+					<mesh filename="package://vulcano_base_description/meshes/wheels/wheel_1.dae" />
+				</xacro:unless>
           </geometry>
         </xacro:if>
@@ -44,5 +108,5 @@
       </visual>
       <collision>
-				<origin xyz="0 0 0" rpy="${M_PI/2} 0 0" />
+		<origin xyz="0 0 0" rpy="${M_PI/2} 0 0" />
         <geometry>
           <cylinder length="${wheel_height}" radius="${wheel_radius}" />
@@ -54,23 +118,32 @@
         <cylinder_inertia  m="${wheel_mass}" r="${wheel_radius}" h="${wheel_height}" />
       </inertial>
-    </link>
-    <!-- Transmission is important to link the joints and the controller (see summit_xl_control/config/summit_xl_control.yaml)-->
+   </link>
+   <!--WHEEL TIRE -->
+    <joint name="joint_${name}_wheel" type="continuous">
+      <parent link="${name}_motor_wheel"/>
+      <child link="${name}_wheel"/>
+      <origin xyz="0 0 0" rpy="0 0 ${M_PI}" />
+      <axis xyz="0 1 0" rpy="0 0 0" />
+      <limit effort="${wheel_joint_effort_limit}" velocity="${wheel_joint_velocity_limit}"/>
+      <joint_properties damping="${wheel_joint_damping}" friction="{wheel_joint_friction}"/>
+    </joint>
     <transmission name="${name}_wheel_joint_trans">
       <type>transmission_interface/SimpleTransmission</type>
       <joint name="joint_${name}_wheel">
-		<hardwareInterface>EffortJointInterface</hardwareInterface>
+		<!-- hardwareInterface>EffortJointInterface</hardwareInterface -->
+		<hardwareInterface>VelocityJointInterface</hardwareInterface>
       </joint>
       <actuator name="${name}_wheel_joint_motor">
-        <mechanicalReduction>1</mechanicalReduction>
+        <mechanicalReduction>${wheel_mechanical_reduction}</mechanicalReduction>
       </actuator>
      </transmission>
-    <gazebo reference="${name}_wheel">
-			<mu1 value="1.0"/>
-			<mu2 value="1.0"/>
-			<kp value="10000000.0" />
-			<kd value="1.0" />
-			<fdir1 value="1 0 0"/>
-      <turnGravityOff>false</turnGravityOff>
-    </gazebo>
+   <gazebo reference="${name}_wheel">
+		<mu1 value="1.0"/>
+		<mu2 value="1.0"/>
+		<kp value="10000000.0" />
+		<kd value="1.0" />
+		<fdir1 value="1 0 0"/>
+        <turnGravityOff>false</turnGravityOff>
+   </gazebo>
   </xacro:macro>
 </robot>

Commit message: modified hardwareInterface from motorwheel to EffortJointInterface - that works better from plugin

File: vulcano_base_description/robots/vulcano_base.urdf.xacro (robot description, xacro)
@@ -31,4 +31,5 @@
   <!-- Gazebo omni steering plugin -->
   <!-- xacro:omni_steering/ -->
+  <xacro:omni_drive/>
   <xacro:motor_wheel name="front_right" parent="base_link" reflect="false" hq="true">
 	<origin xyz="${wheel_offset_x} -${wheel_offset_y} ${wheel_offset_z}" rpy="0 0 0"/>
@@ -49,7 +50,7 @@
 	 <origin xyz="0.0 0.0 0.33" rpy="0 0 0"/>
   </xacro:sensor_hokuyo_utm30lx>
-  <xacro:sensor_axis name="camera" parent="base_link">
+  <!-- xacro:sensor_axis name="camera" parent="base_link">
 	<origin xyz="0.19 0 0.17" rpy="0 ${15*PI/180} 0"/>
-  </xacro:sensor_axis>
+  </xacro:sensor_axis -->
   <xacro:sensor_imu name="imu" parent="base_link">
 	<origin xyz="-0.18 0.0 0.170" rpy="0 0 0"/>

File: vulcano_base_description/urdf/bases/vulcano_base.gazebo.xacro (robot description, xacro)
@@ -23,4 +23,23 @@
 	  </gazebo>
   </xacro:macro>
+  <xacro:macro name="omni_drive">
+		<gazebo>
+		<plugin name="omni_drive" filename="libomnidrive_plugin.so">
+			<robotNamespace>/vulcano_base</robotNamespace>
+			<robotParam>robot_description</robotParam>
+			<broadcastTF>1</broadcastTF>
+			<wheelDiameter>0.15</wheelDiameter>
+			<wheelBase>0.933</wheelBase>
+			<trackWidth>0.57</trackWidth>
+			<wheelTorque>40.0</wheelTorque>
+			<motorWheelTorque>25.0</motorWheelTorque>
+			<commandTopic>/vulcano_base_control/cmd_vel</commandTopic>
+			<odometryTopic>/vulcano_base/odom</odometryTopic>
+			<odometryFrame>odom</odometryFrame>
+			<robotBaseFrame>base_footprint</robotBaseFrame>
+			<updateRate>100.0</updateRate>
+		</plugin>
+		</gazebo>
+  </xacro:macro>
   <gazebo reference="base_footprint">
     <material>Gazebo/Green</material>

File: vulcano_base_description/urdf/bases/vulcano_base.urdf.xacro (robot description, xacro)
@@ -27,5 +27,5 @@
       <mass value="25.0" />
       <origin xyz="0 0 0" />
-      <inertia  ixx="1.391" ixy="0.004"  ixz="0.0"  iyy="6.853"  iyz="0.0"  izz="6.125" />
+      <inertia  ixx="1.0" ixy="0.0"  ixz="0.0"  iyy="1.0"  iyz="0.0"  izz="1.0" />
     </inertial>
     <visual>
@@ -38,5 +38,5 @@
        <xacro:unless value="${hq}">
        <geometry>
-	     <mesh filename="package://vulcano_base_description/meshes/bases/vulcano_base_chassis.stl"/>
+	     <mesh filename="package://vulcano_base_description/meshes/bases/vulcano_base_chassis.dae"/>
        </geometry>
        </xacro:unless>
@@ -56,5 +56,5 @@
       <mass value="15.0" />
       <origin xyz="0 0 0" />
-      <inertia  ixx="1.391" ixy="0.004"  ixz="0.0"  iyy="6.853"  iyz="0.0"  izz="6.125" />
+      <inertia  ixx="0.1" ixy="0.0"  ixz="0.0"  iyy="0.1"  iyz="0.0"  izz="0.1" />
     </inertial>
     <visual>
@@ -67,5 +67,5 @@
        <xacro:unless value="${hq}">
        <geometry>
-	     <mesh filename="package://vulcano_base_description/meshes/bases/vulcano_base_cabinet.stl"/>
+	     <mesh filename="package://vulcano_base_description/meshes/bases/vulcano_base_cabinet.dae"/>
        </geometry>
        </xacro:unless>

File: vulcano_base_description/urdf/wheels/motor_wheel.urdf.xacro (robot description, xacro)
@@ -5,5 +5,5 @@
   <property name="wheel_radius" value="0.093" />
   <property name="wheel_height" value="0.14" />
-  <property name="wheel_mass" value="6.5" /> <!-- in kg-->
+  <property name="wheel_mass" value="5.0" /> <!-- in kg-->
   <xacro:property name="steer_joint_damping" value="2.0" />
   <xacro:property name="steer_joint_friction" value="1.0" />
@@ -11,6 +11,6 @@
   <xacro:property name="steer_joint_velocity_limit" value="100.0" />
   <xacro:property name="motor_wheel_mechanical_reduction" value="100.0" />
-  <xacro:property name="wheel_joint_damping" value="1.0" />
-  <xacro:property name="wheel_joint_friction" value="1.0" />
+  <xacro:property name="wheel_joint_damping" value="0.1" />
+  <xacro:property name="wheel_joint_friction" value="0.1" />
   <xacro:property name="wheel_joint_effort_limit" value="1000.0" />
   <xacro:property name="wheel_joint_velocity_limit" value="2000.0" />
@@ -62,5 +62,5 @@
       </collision>
       <inertial>
-        <mass value="20" />
+        <mass value="10" />
         <origin xyz="0 0 0" />
 		<inertia  ixx="0.01" ixy="0.0"  ixz="0.0"  iyy="0.01"  iyz="0.0"  izz="0.01" />
@@ -110,5 +110,6 @@
 		<origin xyz="0 0 0" rpy="${M_PI/2} 0 0" />
         <geometry>
-          <cylinder length="${wheel_height}" radius="${wheel_radius}" />
+          <!-- cylinder length="${wheel_height}" radius="${wheel_radius}" / -->
+          <sphere radius="${wheel_radius}" />
         </geometry>
       </collision>
@@ -131,6 +132,6 @@
       <type>transmission_interface/SimpleTransmission</type>
       <joint name="joint_${name}_wheel">
-		<!-- hardwareInterface>EffortJointInterface</hardwareInterface -->
-		<hardwareInterface>VelocityJointInterface</hardwareInterface>
+		<hardwareInterface>EffortJointInterface</hardwareInterface>
+		<!-- hardwareInterface>VelocityJointInterface</hardwareInterface -->
       </joint>
       <actuator name="${name}_wheel_joint_motor">
@@ -138,5 +139,5 @@
       </actuator>
      </transmission>
-   <gazebo reference="${name}_wheel">
+   <!-- gazebo reference="${name}_wheel">
 		<mu1 value="1.0"/>
 		<mu2 value="1.0"/>
@@ -145,5 +146,5 @@
 		<fdir1 value="1 0 0"/>
         <turnGravityOff>false</turnGravityOff>
-   </gazebo>
+   </gazebo -->
   </xacro:macro>
 </robot>
