Commit message: vulcano_base_common: updated urdf and set namespace to vulcano

File: vulcano_base_description/robots/vulcano_base_standalone.urdf.xacro (robot description, xacro)
@@ -12,4 +12,4 @@
     <xacro:property name="hq" value="true" />
     <xacro:vulcano_base prefix="${prefix}" publish_bf="${publish_bf}" hq="${hq}"/>
-    <xacro:ros_control ns="/vulcano_base"/>
+    <xacro:ros_control ns="/vulcano"/>
 </robot>

File: vulcano_base_description/urdf/vulcano_base.urdf.xacro (robot description, xacro)
@@ -44,12 +44,4 @@
         </xacro:motor_wheel>
         <!-- SENSORS see robotnik_sensors for the specific configuration -->
-        <!-- Hokuyo laser sensors can be parametized with min_angle and max_angle e.g: -->
-        <!--xacro:sensor_hokuyo_utm30lx name="hokuyo_base" parent="base_link" min_angle="2.35" max_angle="-2.35"-->
-        <xacro:sensor_hokuyo_utm30lx name="hokuyo_base" parent="${prefix}base_link">
-           <origin xyz="0.0 0.0 0.33" rpy="0 0 0"/>
-        </xacro:sensor_hokuyo_utm30lx>
-        <!-- xacro:sensor_axis name="camera" parent="${prefix}base_link">
-          <origin xyz="0.19 0 0.17" rpy="0 ${15*PI/180} 0"/>
-        </xacro:sensor_axis -->
         <xacro:sensor_imu name="imu" parent="${prefix}base_link">
           <origin xyz="-0.18 0.0 0.170" rpy="0 0 0"/>
@@ -61,14 +53,4 @@
             <origin xyz="-0.606321 -0.345821 0.3095" rpy="${180*deg2rad} 0 ${235*deg2rad}"/>
         </xacro:sensor_sick_s300>
-        <!--
-            <xacro:sensor_kinect name="kinect" parent="${prefix}base_link">
-                <origin xyz="0.325 0.0 0.16" rpy="0 0 0"/>
-            </xacro:sensor_kinect>
-        -->
-        <!--
-            <xacro:sensor_fotonic name="fotonic" parent="${prefix}base_link">
-                <origin xyz="0.3 0.0 0.24" rpy="0 0 0"/>
-            </xacro:sensor_fotonic>
-        -->
    </xacro:macro>
 </robot>

Commit message: vulcano_base_description: corrected wheel orientations

File: vulcano_base_description/robots/vulcano_base_standalone.urdf.xacro (robot description, xacro)
@@ -12,4 +12,4 @@
     <xacro:property name="hq" value="true" />
     <xacro:vulcano_base prefix="${prefix}" publish_bf="${publish_bf}" hq="${hq}"/>
-    <xacro:ros_control ns="/vulcano"/>
+    <xacro:ros_control />
 </robot>

File: vulcano_base_description/urdf/bases/base.gazebo.xacro (robot description, xacro)
@@ -27,4 +27,5 @@
 			<odometryTopic>odom</odometryTopic>
 			<odometryFrame>odom</odometryFrame>
+			<odometrySource>encoder</odometrySource>
 			<robotBaseFrame>base_footprint</robotBaseFrame>
 			<updateRate>100.0</updateRate>

File: vulcano_base_description/urdf/common.gazebo.xacro (robot description, xacro)
@@ -2,5 +2,5 @@
 <robot xmlns:xacro="http://ros.org/wiki/xacro">
   <!-- ros control plugin -->
-  <xacro:macro name="ros_control" params="ns">
+  <xacro:macro name="ros_control" > <!--  params="ns"  -->
     <gazebo>
       <plugin name="ros_control" filename="libgazebo_ros_control.so">

File: vulcano_base_description/urdf/vulcano_base.urdf.xacro (robot description, xacro)
@@ -34,11 +34,11 @@
           <origin xyz="${wheel_offset_x} -${wheel_offset_y} ${wheel_offset_z}" rpy="0 0 0"/>
         </xacro:motor_wheel>
-        <xacro:motor_wheel prefix="${prefix}front_left_" parent="${prefix}base_link" reflect="true" hq="true">
-          <origin xyz="${wheel_offset_x} ${wheel_offset_y} ${wheel_offset_z}" rpy="0 0 0"/>
+        <xacro:motor_wheel prefix="${prefix}front_left_" parent="${prefix}base_link" reflect="false" hq="true">
+          <origin xyz="${wheel_offset_x} ${wheel_offset_y} ${wheel_offset_z}" rpy="0 0 ${180.0*deg2rad}"/>
         </xacro:motor_wheel>
         <xacro:motor_wheel prefix="${prefix}back_left_" parent="${prefix}base_link" reflect="false" hq="true">
-          <origin xyz="-${wheel_offset_x} ${wheel_offset_y} ${wheel_offset_z}" rpy="0 0 0"/>
+          <origin xyz="-${wheel_offset_x} ${wheel_offset_y} ${wheel_offset_z}" rpy="0 0 ${180.0*deg2rad}"/>
         </xacro:motor_wheel>
-        <xacro:motor_wheel prefix="${prefix}back_right_" parent="${prefix}base_link" reflect="true" hq="true">
+        <xacro:motor_wheel prefix="${prefix}back_right_" parent="${prefix}base_link" reflect="false" hq="true">
           <origin xyz="-${wheel_offset_x} -${wheel_offset_y} ${wheel_offset_z}" rpy="0 0 0"/>
         </xacro:motor_wheel>

File: vulcano_base_description/urdf/wheels/motor_wheel.urdf.xacro (robot description, xacro)
@@ -22,11 +22,12 @@
   </xacro:macro>
   <xacro:macro name="motor_wheel" params="prefix parent *origin reflect hq">
+  <!-- TODO: check reflect parameter -->
   <!--MOTOR WHEEL -->
-    <joint name="${prefix}motor_wheel_joint" type="continuous">
+    <joint name="${prefix}motor_wheel_joint" type="revolute">
       <parent link="${parent}"/>
       <child link="${prefix}motor_wheel"/>
       <insert_block name="origin" />
       <axis xyz="0 0 1" rpy="0 0 0" />
-      <!-- limit effort="${steer_joint_effort_limit}" velocity="${steer_joint_velocity_limit}" lower="-1.5708" upper="1.5708"/ -->
+      <!-- limit effort="${steer_joint_effort_limit}" velocity="${steer_joint_velocity_limit}" lower="-1.5708" upper="1.5708" / -->
       <limit effort="${steer_joint_effort_limit}" velocity="${steer_joint_velocity_limit}" lower="-3.00" upper="3.00"/>
       <joint_properties damping="${steer_joint_damping}" friction="{steer_joint_friction}"/>
