Commit message: Added modularized models

File: vulcano_base_description/urdf/bases/base.gazebo.xacro (robot description, xacro)
@@ -1,18 +1,8 @@
 <?xml version="1.0"?>
 <robot xmlns:xacro="http://ros.org/wiki/xacro">
-  <!-- ros control plugin -->
-  <xacro:macro name="ros_control">
-    <gazebo>
-      <plugin name="ros_control" filename="libgazebo_ros_control.so">
-        <robotNamespace>/vulcano_base</robotNamespace>
-        <robotParam>robot_description</robotParam>
-        <controlPeriod>0.001</controlPeriod>
-	    <robotSimType>gazebo_ros_control/DefaultRobotHWSim</robotSimType>
-      </plugin>
-    </gazebo>
-	</xacro:macro>
   <xacro:macro name="omni_steering">
 		<gazebo>
 	    <plugin name="omni_steering" filename="libgazebo_ros_planar_move.so">
+		  <robotNamespace>/vulcano_base</robotNamespace>
 	      <commandTopic>/vulcano_base_control/cmd_vel</commandTopic>
 	      <odometryTopic>/vulcano_base/odom</odometryTopic>
@@ -29,16 +19,14 @@
 			<robotParam>robot_description</robotParam>
 			<broadcastTF>1</broadcastTF>
-			<wheelDiameter>0.186</wheelDiameter>
-			<wheelBase>0.934</wheelBase>
+			<wheelDiameter>0.15</wheelDiameter>
+			<wheelBase>0.933</wheelBase>
 			<trackWidth>0.57</trackWidth>
 			<wheelTorque>40.0</wheelTorque>
 			<motorWheelTorque>25.0</motorWheelTorque>
-			<commandTopic>/vulcano_base_control/cmd_vel</commandTopic>
+			<commandTopic>/vulcano_base_control/cmd_vel</commandTopic>  <!-- TODO: review topics -->
 			<odometryTopic>/vulcano_base/odom</odometryTopic>
 			<odometryFrame>odom</odometryFrame>
 			<robotBaseFrame>base_footprint</robotBaseFrame>
 			<updateRate>100.0</updateRate>
-			<odometrySource>encoder</odometrySource>
-			<mirrored_axes>false</mirrored_axes>
 		</plugin>
 		</gazebo>

File: vulcano_base_description/urdf/bases/base.urdf.xacro (robot description, xacro)
@@ -1,6 +1,5 @@
 <?xml version="1.0"?>
-<robot name="vulcano_base" xmlns:xacro="http://www.ros.org/wiki/xacro">
-  <xacro:include filename="$(find vulcano_base_description)/urdf/bases/vulcano_base.gazebo.xacro" />
-  <xacro:macro name="vulcano_base" params="name publish_bf hq">
+<robot xmlns:xacro="http://www.ros.org/wiki/xacro">
+  <xacro:macro name="base" params="prefix publish_bf hq">
   <!-- Robot mechanical and motor parameters -->
   <xacro:property name="PI" value="3.1415926535897931"/>
@@ -8,5 +7,5 @@
   <!-- BASE FOOTPRINT -->
   <xacro:if value="${publish_bf}">
-    <link name="base_footprint">
+    <link name="${prefix}base_footprint">
       <visual>
           <origin xyz="0 0 0" rpy="0 0 0" />
@@ -18,10 +17,10 @@
     <joint name="base_footprint_joint" type="fixed">
       <origin xyz="0 0 ${wheel_radius}" rpy="0 0 0" /> <!-- ${wheel_radius} property must be defined inside wheel description -->
-      <parent link="base_footprint"/>
-      <child link="base_link" />
+      <parent link="${prefix}base_footprint"/>
+      <child link="${prefix}base_link" />
     </joint>
   </xacro:if>
   <!-- BASE_LINK -->
-  <link name="base_link">
+  <link name="${prefix}base_link">
     <inertial>
       <mass value="25.0" />
@@ -52,5 +51,5 @@
     </collision>
   </link>
-  <link name="cabinet_link">
+  <link name="${prefix}cabinet_link">
     <inertial>
       <mass value="15.0" />
@@ -81,8 +80,8 @@
     </collision>
   </link>
-  <joint name="cabinet_joint" type="fixed">
+  <joint name="${prefix}cabinet_joint" type="fixed">
     <origin xyz="0 0 0.234" rpy="0 0 0" />
-    <parent link="base_link"/>
-    <child link="cabinet_link" />
+    <parent link="${prefix}base_link"/>
+    <child link="${prefix}cabinet_link" />
   </joint>
   </xacro:macro>

File: vulcano_base_description/urdf/wheels/motor_wheel.urdf.xacro (robot description, xacro)
@@ -1,4 +1,4 @@
 <?xml version="1.0"?>
-<robot name="wheel" xmlns:xacro="http://www.ros.org/wiki/xacro">
+<robot xmlns:xacro="http://www.ros.org/wiki/xacro">
   <xacro:property name="M_PI" value="3.1415926535897931" />
   <!-- Wheels -->
@@ -21,7 +21,25 @@
               izz="${m*r*r/2}" />
   </xacro:macro>
-  <xacro:macro name="motor_wheel" params="name parent *origin reflect hq">
+  <xacro:macro name="motor_wheel" params="prefix parent *origin reflect hq">
   <!--MOTOR WHEEL -->
-  <link name="${name}_motor_wheel">
+    <joint name="${prefix}motor_wheel_joint" type="continuous">
+      <parent link="${parent}"/>
+      <child link="${prefix}motor_wheel"/>
+      <insert_block name="origin" />
+      <axis xyz="0 0 1" rpy="0 0 0" />
+      <!-- limit effort="${steer_joint_effort_limit}" velocity="${steer_joint_velocity_limit}" lower="-1.5708" upper="1.5708"/ -->
+      <limit effort="${steer_joint_effort_limit}" velocity="${steer_joint_velocity_limit}" lower="-3.00" upper="3.00"/>
+      <joint_properties damping="${steer_joint_damping}" friction="{steer_joint_friction}"/>
+    </joint>
+  <transmission name="${prefix}motor_wheel_trans">
+     <type>transmission_interface/SimpleTransmission</type>
+     <joint name="${prefix}motor_wheel_joint">
+        <hardwareInterface>EffortJointInterface</hardwareInterface>
+     </joint>
+     <actuator name="${prefix}motor_wheel_motor">
+        <mechanicalReduction>${motor_wheel_mechanical_reduction}</mechanicalReduction>
+     </actuator>
+  </transmission>
+  <link name="${prefix}motor_wheel">
       <visual>
         <!-- HIGH RESOLUTION WHEELS -->
@@ -29,10 +47,10 @@
           <origin xyz="0 0 0" rpy="0 0 0" />
           <geometry>
-				<xacro:if value="${reflect}">
-					<mesh filename="package://vulcano_base_description/meshes/wheels/motorwheel_2.dae" />
-				</xacro:if>
-				<xacro:unless value="${reflect}">
-					<mesh filename="package://vulcano_base_description/meshes/wheels/motorwheel_2.dae" />
-				</xacro:unless>
+                <xacro:if value="${reflect}">
+                    <mesh filename="package://vulcano_base_description/meshes/wheels/motorwheel_2.dae" />
+                </xacro:if>
+                <xacro:unless value="${reflect}">
+                    <mesh filename="package://vulcano_base_description/meshes/wheels/motorwheel_2.dae" />
+                </xacro:unless>
           </geometry>
         </xacro:if>
@@ -41,22 +59,22 @@
           <origin xyz="0 0 0" rpy="0 0 0" />
           <geometry>
-				<xacro:if value="${reflect}">
-					<mesh filename="package://vulcano_base_description/meshes/wheels/motorwheel_2.stl" />
-				</xacro:if>
-				<xacro:unless value="${reflect}">
-					<mesh filename="package://vulcano_base_description/meshes/wheels/motorwheel_2.stl" />
-				</xacro:unless>
+                <xacro:if value="${reflect}">
+                    <mesh filename="package://vulcano_base_description/meshes/wheels/motorwheel_2.stl" />
+                </xacro:if>
+                <xacro:unless value="${reflect}">
+                    <mesh filename="package://vulcano_base_description/meshes/wheels/motorwheel_2.stl" />
+                </xacro:unless>
           </geometry>
         </xacro:unless>
       </visual>
       <collision>
-		<origin xyz="0 0 0" rpy="0 0 0" />
+        <origin xyz="0 0 0" rpy="0 0 0" />
         <geometry>
-				<xacro:if value="${reflect}">
-					<mesh filename="package://vulcano_base_description/meshes/wheels/motorwheel_2.dae" />
-				</xacro:if>
-				<xacro:unless value="${reflect}">
-					<mesh filename="package://vulcano_base_description/meshes/wheels/motorwheel_2.dae" />
-				</xacro:unless>
+                <xacro:if value="${reflect}">
+                    <mesh filename="package://vulcano_base_description/meshes/wheels/motorwheel_2.dae" />
+                </xacro:if>
+                <xacro:unless value="${reflect}">
+                    <mesh filename="package://vulcano_base_description/meshes/wheels/motorwheel_2.dae" />
+                </xacro:unless>
         </geometry>
       </collision>
@@ -64,26 +82,27 @@
         <mass value="10" />
         <origin xyz="0 0 0" />
-		<inertia  ixx="0.01" ixy="0.0"  ixz="0.0"  iyy="0.01"  iyz="0.0"  izz="0.01" />
-	  </inertial>
+        <inertia  ixx="0.01" ixy="0.0"  ixz="0.0"  iyy="0.01"  iyz="0.0"  izz="0.01" />
+      </inertial>
     </link>
-    <joint name="joint_${name}_motor_wheel" type="continuous">
-      <parent link="${parent}"/>
-      <child link="${name}_motor_wheel"/>
-      <insert_block name="origin" />
-      <axis xyz="0 0 1" rpy="0 0 0" />
-      <!-- limit effort="${steer_joint_effort_limit}" velocity="${steer_joint_velocity_limit}" lower="-1.5708" upper="1.5708"/ -->
-      <limit effort="${steer_joint_effort_limit}" velocity="${steer_joint_velocity_limit}" lower="-3.00" upper="3.00"/>
-      <joint_properties damping="${steer_joint_damping}" friction="{steer_joint_friction}"/>
+   <!--WHEEL TIRE -->
+   <joint name="${prefix}wheel_joint" type="continuous">
+        <parent link="${prefix}motor_wheel"/>
+        <child link="${prefix}wheel"/>
+        <origin xyz="0 0 0" rpy="0 0 ${M_PI}" />
+        <axis xyz="0 1 0" rpy="0 0 0" />
+        <limit effort="${wheel_joint_effort_limit}" velocity="${wheel_joint_velocity_limit}"/>
+        <joint_properties damping="${wheel_joint_damping}" friction="{wheel_joint_friction}"/>
     </joint>
-  <transmission name="${name}_motor_wheel_joint_trans">
-	 <type>transmission_interface/SimpleTransmission</type>
-     <joint name="joint_${name}_motor_wheel">
-		<hardwareInterface>EffortJointInterface</hardwareInterface>
+    <transmission name="${prefix}wheel_trans">
+     <type>transmission_interface/SimpleTransmission</type>
+     <joint name="${prefix}wheel_joint">
+       <hardwareInterface>EffortJointInterface</hardwareInterface>
+        <!--<hardwareInterface>VelocityJointInterface</hardwareInterface>-->
      </joint>
-     <actuator name="${name}_motor_wheel_joint_motor">
-        <mechanicalReduction>${motor_wheel_mechanical_reduction}</mechanicalReduction>
+     <actuator name="${prefix}wheel_motor">
+       <mechanicalReduction>${wheel_mechanical_reduction}</mechanicalReduction>
      </actuator>
-  </transmission>
-  <link name="${name}_wheel">
+    </transmission>
+  <link name="${prefix}wheel">
       <visual>
         <!-- HIGH RESOLUTION WHEELS -->
@@ -91,10 +110,10 @@
           <origin xyz="0 0 0" rpy="0 0 0" />
           <geometry>
-				<xacro:if value="${reflect}">
-					<mesh filename="package://vulcano_base_description/meshes/wheels/wheel_1.dae" />
-				</xacro:if>
-				<xacro:unless value="${reflect}">
-					<mesh filename="package://vulcano_base_description/meshes/wheels/wheel_1.dae" />
-				</xacro:unless>
+                <xacro:if value="${reflect}">
+                    <mesh filename="package://vulcano_base_description/meshes/wheels/wheel_1.dae" />
+                </xacro:if>
+                <xacro:unless value="${reflect}">
+                    <mesh filename="package://vulcano_base_description/meshes/wheels/wheel_1.dae" />
+                </xacro:unless>
           </geometry>
         </xacro:if>
@@ -108,5 +127,5 @@
       </visual>
       <collision>
-		<origin xyz="0 0 0" rpy="${M_PI/2} 0 0" />
+        <origin xyz="0 0 0" rpy="${M_PI/2} 0 0" />
         <geometry>
           <!-- cylinder length="${wheel_height}" radius="${wheel_radius}" / -->
@@ -120,29 +139,10 @@
       </inertial>
    </link>
-   <!--WHEEL TIRE -->
-    <joint name="joint_${name}_wheel" type="continuous">
-      <parent link="${name}_motor_wheel"/>
-      <child link="${name}_wheel"/>
-      <origin xyz="0 0 0" rpy="0 0 ${M_PI}" />
-      <axis xyz="0 1 0" rpy="0 0 0" />
-      <limit effort="${wheel_joint_effort_limit}" velocity="${wheel_joint_velocity_limit}"/>
-      <joint_properties damping="${wheel_joint_damping}" friction="{wheel_joint_friction}"/>
-    </joint>
-    <transmission name="${name}_wheel_joint_trans">
-      <type>transmission_interface/SimpleTransmission</type>
-      <joint name="joint_${name}_wheel">
-		<hardwareInterface>EffortJointInterface</hardwareInterface>
-		<!-- hardwareInterface>VelocityJointInterface</hardwareInterface -->
-      </joint>
-      <actuator name="${name}_wheel_joint_motor">
-        <mechanicalReduction>${wheel_mechanical_reduction}</mechanicalReduction>
-      </actuator>
-     </transmission>
-   <!-- gazebo reference="${name}_wheel">
-		<mu1 value="1.0"/>
-		<mu2 value="1.0"/>
-		<kp value="10000000.0" />
-		<kd value="1.0" />
-		<fdir1 value="1 0 0"/>
+   <!-- gazebo reference="${prefix}wheel">
+        <mu1 value="1.0"/>
+        <mu2 value="1.0"/>
+        <kp value="10000000.0" />
+        <kd value="1.0" />
+        <fdir1 value="1 0 0"/>
         <turnGravityOff>false</turnGravityOff>
    </gazebo -->
