Commit message: vulcano_base_description: changed collision model of motorwheel

File: vulcano_base_description/urdf/wheels/motor_wheel.urdf.xacro (robot description, xacro)
@@ -130,6 +130,12 @@
         <origin xyz="0 0 0" rpy="${M_PI/2} 0 0" />
         <geometry>
+          <xacro:if value="${reflect}">
+              <mesh filename="package://vulcano_base_description/meshes/wheels/wheel_1.dae" />
+          </xacro:if>
+          <xacro:unless value="${reflect}">
+              <mesh filename="package://vulcano_base_description/meshes/wheels/wheel_1.dae" />
+          </xacro:unless>
           <!-- cylinder length="${wheel_height}" radius="${wheel_radius}" / -->
-          <sphere radius="${wheel_radius}" />
+          <!--<sphere radius="${wheel_radius}" />-->
         </geometry>
       </collision>

Commit message: vulcano_base_description: updated wheel limits

File: vulcano_base_description/urdf/wheels/motor_wheel.urdf.xacro (robot description, xacro)
@@ -9,6 +9,6 @@
   <xacro:property name="steer_joint_friction" value="1.0" />
   <xacro:property name="steer_joint_effort_limit" value="100.0" />
-  <xacro:property name="steer_joint_velocity_limit" value="100.0" />
-  <xacro:property name="motor_wheel_mechanical_reduction" value="100.0" />
+  <xacro:property name="steer_joint_velocity_limit" value="0.6" />
+  <xacro:property name="motor_wheel_mechanical_reduction" value="1.0" />
   <xacro:property name="wheel_joint_damping" value="0.1" />
   <xacro:property name="wheel_joint_friction" value="0.1" />

Commit message: vulcano_base_description: updated wheel limits

File: vulcano_base_description/urdf/wheels/motor_wheel.urdf.xacro (robot description, xacro)
@@ -9,6 +9,7 @@
   <xacro:property name="steer_joint_friction" value="1.0" />
   <xacro:property name="steer_joint_effort_limit" value="100.0" />
-  <xacro:property name="steer_joint_velocity_limit" value="100.0" />
-  <xacro:property name="motor_wheel_mechanical_reduction" value="100.0" />
+  <xacro:property name="steer_joint_velocity_limit" value="2" />
+  <xacro:property name="steer_joint_position_limit" value="2.8" />
+  <xacro:property name="motor_wheel_mechanical_reduction" value="1.0" />
   <xacro:property name="wheel_joint_damping" value="0.1" />
   <xacro:property name="wheel_joint_friction" value="0.1" />
@@ -29,6 +30,5 @@
       <insert_block name="origin" />
       <axis xyz="0 0 1" rpy="0 0 0" />
-      <!-- limit effort="${steer_joint_effort_limit}" velocity="${steer_joint_velocity_limit}" lower="-1.5708" upper="1.5708" / -->
-      <limit effort="${steer_joint_effort_limit}" velocity="${steer_joint_velocity_limit}" lower="-3.00" upper="3.00"/>
+      <limit effort="${steer_joint_effort_limit}" velocity="${steer_joint_velocity_limit}" lower="-${steer_joint_position_limit}" upper="${steer_joint_position_limit}"/>
       <joint_properties damping="${steer_joint_damping}" friction="${steer_joint_friction}"/>
     </joint>
