Commit message: added sick s300 lasers to model

File: vulcano_base_description/urdf/vulcano_base.urdf.xacro (robot description, xacro)
@@ -16,4 +16,5 @@
     <!-- ***************** -->
     <xacro:property name="PI" value="3.1415926535897931"/>
+    <xacro:property name="deg2rad" value="0.01745329251"/>
     <!-- Wheel parameters -->
     <xacro:property name="wheel_offset_x" value="0.467" />    <!-- x,y,z in translation from base_link to the center of the wheel -->
@@ -54,4 +55,10 @@
           <origin xyz="-0.18 0.0 0.170" rpy="0 0 0"/>
         </xacro:sensor_imu>
+        <xacro:sensor_sick_s300 name="front_left" parent="${prefix}base_link">
+            <origin xyz="0.606321 0.345821 0.3095" rpy="${180*deg2rad} 0 ${45*deg2rad}"/>
+        </xacro:sensor_sick_s300>
+        <xacro:sensor_sick_s300 name="back_right" parent="${prefix}base_link">
+            <origin xyz="-0.606321 -0.345821 0.3095" rpy="${180*deg2rad} 0 ${235*deg2rad}"/>
+        </xacro:sensor_sick_s300>
         <!--
             <xacro:sensor_kinect name="kinect" parent="${prefix}base_link">

Commit message: vulcano_base_description: corrected ros_control interfaces on xacro files

File: vulcano_base_description/urdf/vulcano_base.urdf.xacro (robot description, xacro)
@@ -28,7 +28,4 @@
     <xacro:macro name="vulcano_base" params="prefix publish_bf hq">
         <xacro:base prefix="${prefix}" publish_bf="${publish_bf}" hq="${hq}"/>
-        <!-- Gazebo omni steering plugin -->
-        <!--<xacro:omni_steering/>-->
-        <xacro:omni_drive />
         <xacro:motor_wheel prefix="${prefix}front_right_" parent="${prefix}base_link" reflect="false" hq="true">
           <origin xyz="${wheel_offset_x} -${wheel_offset_y} ${wheel_offset_z}" rpy="0 0 0"/>

File: vulcano_base_description/urdf/wheels/motor_wheel.urdf.xacro (robot description, xacro)
@@ -31,12 +31,13 @@
       <!-- limit effort="${steer_joint_effort_limit}" velocity="${steer_joint_velocity_limit}" lower="-1.5708" upper="1.5708" / -->
       <limit effort="${steer_joint_effort_limit}" velocity="${steer_joint_velocity_limit}" lower="-3.00" upper="3.00"/>
-      <joint_properties damping="${steer_joint_damping}" friction="{steer_joint_friction}"/>
+      <joint_properties damping="${steer_joint_damping}" friction="${steer_joint_friction}"/>
     </joint>
   <transmission name="${prefix}motor_wheel_trans">
      <type>transmission_interface/SimpleTransmission</type>
      <joint name="${prefix}motor_wheel_joint">
-        <hardwareInterface>EffortJointInterface</hardwareInterface>
+        <hardwareInterface>PositionJointInterface</hardwareInterface>
      </joint>
      <actuator name="${prefix}motor_wheel_motor">
+        <hardwareInterface>PositionActuatorInterface</hardwareInterface>
         <mechanicalReduction>${motor_wheel_mechanical_reduction}</mechanicalReduction>
      </actuator>
@@ -98,8 +99,8 @@
      <type>transmission_interface/SimpleTransmission</type>
      <joint name="${prefix}wheel_joint">
-       <hardwareInterface>EffortJointInterface</hardwareInterface>
-        <!--<hardwareInterface>VelocityJointInterface</hardwareInterface>-->
+        <hardwareInterface>VelocityJointInterface</hardwareInterface>
      </joint>
      <actuator name="${prefix}wheel_motor">
+       <hardwareInterface>VelocityActuatorInterface</hardwareInterface>
        <mechanicalReduction>${wheel_mechanical_reduction}</mechanicalReduction>
      </actuator>
@@ -130,12 +131,12 @@
         <origin xyz="0 0 0" rpy="${M_PI/2} 0 0" />
         <geometry>
-          <xacro:if value="${reflect}">
-              <mesh filename="package://vulcano_base_description/meshes/wheels/wheel_1.dae" />
-          </xacro:if>
-          <xacro:unless value="${reflect}">
-              <mesh filename="package://vulcano_base_description/meshes/wheels/wheel_1.dae" />
-          </xacro:unless>
+          <!--<xacro:if value="${reflect}">-->
+              <!--<mesh filename="package://vulcano_base_description/meshes/wheels/wheel_1.dae" />-->
+          <!--</xacro:if>-->
+          <!--<xacro:unless value="${reflect}">-->
+              <!--<mesh filename="package://vulcano_base_description/meshes/wheels/wheel_1.dae" />-->
+          <!--</xacro:unless>-->
           <!-- cylinder length="${wheel_height}" radius="${wheel_radius}" / -->
-          <!--<sphere radius="${wheel_radius}" />-->
+          <sphere radius="${wheel_radius}" />
         </geometry>
       </collision>

Commit message: vulcano_base_description: corrected laser links

File: vulcano_base_description/urdf/vulcano_base.urdf.xacro (robot description, xacro)
@@ -48,6 +48,12 @@
         </xacro:sensor_sick_s300>
         <xacro:sensor_sick_s300 name="back_right_laser" parent="${prefix}base_link">
-            <origin xyz="-0.606321 -0.345821 0.3095" rpy="${180*deg2rad} 0 ${235*deg2rad}"/>
+            <origin xyz="-0.606321 -0.345821 0.3095" rpy="${180*deg2rad} 0 ${225*deg2rad}"/>
         </xacro:sensor_sick_s300>
+        <joint name="merged_base_laser_joint" type="fixed"> <!-- front and back laser will be merged into this link -->
+            <origin xyz="0 0 0.234" rpy="0 0 0" />
+            <parent link="${prefix}base_link"/>
+            <child link="${prefix}merged_base_laser_link" />
+        </joint>
+        <link name="merged_base_laser_link" />
    </xacro:macro>
 </robot>
